Commit message: CHANGES OF CAMERA NAMES: In order to follow the terminology of the reports and deliverables, we renamed - the endeffector_camera to wrist_camera - the camera_top_left to workspace_camera_right

File: camera_pose_calibration/src/ur10.urdf (robot description, URDF)
Before this commit: robot ur10, 42 links, 41 joints
Links:
- removed link camera_top_left_depth_frame
- removed link camera_top_left_depth_optical_frame
- removed link camera_top_left_link
- removed link camera_top_left_rgb_frame
- removed link camera_top_left_rgb_optical_frame
- removed link endeffector_camera_depth_frame
- removed link endeffector_camera_depth_optical_frame
- removed link endeffector_camera_link
- removed link endeffector_camera_rgb_frame
- removed link endeffector_camera_rgb_optical_frame
- added link workspace_camera_right_depth_frame
- added link workspace_camera_right_depth_optical_frame
- added link workspace_camera_right_link, mass 0.1; collision mesh filename=package://ur10_model/meshes/collision/asus.stl scale=0.001 0.001 0.001; visual mesh filename=package://ur10_model/meshes/visual/asus.stl scale=0.001 0.001 0.001
- added link workspace_camera_right_rgb_frame
- added link workspace_camera_right_rgb_optical_frame
- added link wrist_camera_depth_frame
- added link wrist_camera_depth_optical_frame
- added link wrist_camera_link, mass 0.1; collision mesh filename=package://ur10_model/meshes/collision/asus.stl scale=0.001 0.001 0.001; visual mesh filename=package://ur10_model/meshes/visual/asus.stl scale=0.001 0.001 0.001
- added link wrist_camera_rgb_frame
- added link wrist_camera_rgb_optical_frame
Joints:
- removed joint camera_top_left_base_link_joint
- removed joint camera_top_left_base_link_joint2
- removed joint camera_top_left_base_link_joint3
- removed joint camera_top_left_base_link_joint4
- removed joint camera_top_left_frame_joint
- removed joint endeffector_camera_base_link_joint
- removed joint endeffector_camera_base_link_joint2
- removed joint endeffector_camera_base_link_joint3
- removed joint endeffector_camera_base_link_joint4
- removed joint endeffector_camera_frame_joint
- added joint workspace_camera_right_base_link_joint: type fixed, parent workspace_camera_right_link, child workspace_camera_right_depth_frame, origin xyz=0.0 -0.02 0.0 rpy=0.0 0.0 0.0
- added joint workspace_camera_right_base_link_joint2: type fixed, parent workspace_camera_right_link, child workspace_camera_right_rgb_frame, origin xyz=0.0 -0.045 0.0 rpy=0.0 0.0 0.0
- added joint workspace_camera_right_base_link_joint3: type fixed, parent workspace_camera_right_depth_frame, child workspace_camera_right_depth_optical_frame, origin xyz=0.0 0.0 0.0 rpy=-1.57079632679 0.0 -1.57079632679
- added joint workspace_camera_right_base_link_joint4: type fixed, parent workspace_camera_right_rgb_frame, child workspace_camera_right_rgb_optical_frame, origin xyz=0.0 0.0 0.0 rpy=-1.57079632679 0.0 -1.57079632679
- added joint workspace_camera_right_frame_joint: type fixed, parent front_bar, child workspace_camera_right_link, origin xyz=1.1574900035 0.379638906853 -1.19623791051 rpy=0.224178449253 -0.00758963460292 3.12106772132
- added joint wrist_camera_base_link_joint: type fixed, parent wrist_camera_link, child wrist_camera_depth_frame, origin xyz=0.0 -0.02 0.0 rpy=0.0 0.0 0.0
- added joint wrist_camera_base_link_joint2: type fixed, parent wrist_camera_link, child wrist_camera_rgb_frame, origin xyz=0.0 -0.045 0.0 rpy=0.0 0.0 0.0
- added joint wrist_camera_base_link_joint3: type fixed, parent wrist_camera_depth_frame, child wrist_camera_depth_optical_frame, origin xyz=0.0 0.0 0.0 rpy=-1.57079632679 0.0 -1.57079632679
- added joint wrist_camera_base_link_joint4: type fixed, parent wrist_camera_rgb_frame, child wrist_camera_rgb_optical_frame, origin xyz=0.0 0.0 0.0 rpy=-1.57079632679 0.0 -1.57079632679
- added joint wrist_camera_frame_joint: type fixed, parent wrist_3_link, child wrist_camera_link, origin xyz=0.444859979541 -0.490573541562 0.160347068916 rpy=-1.78497299393 1.48671173388 -1.93695858476
